Commit message: Removed autobot_scan_merger submodule, updated the sensor visualisation in Gazebo

File: src/autobot_description/xacro/autobot_core.xacro (robot description, xacro)
@@ -15,4 +15,5 @@
     <!-- * * * Link Definitions * * * -->
     <link name="base_link"/>
+    <link name="laser_merged" />
     <link name="chassis_lower">
         <visual>
@@ -127,4 +128,9 @@
         <origin xyz="0.0 0.0 ${ground_clearance}" rpy="0.0 0.0 0.0"/>
     </joint>
+    <joint name="chassis_lower_to_laser_merged" type="fixed">
+        <parent link="chassis_lower"/>
+        <child link="laser_merged"/>
+        <origin xyz="0.0 0.0 ${chassis_height/2 - 0.015}" rpy="0.0 0.0 0.0" />
+    </joint>
     <joint name="chassis_lower_to_left_drive_wheel" type="continuous">
         <parent link="chassis_lower"/>

File: src/autobot_description/xacro/sensors.xacro (robot description, xacro)
@@ -29,5 +29,5 @@
             <sensor name="${name}" type="gpu_ray">
                 <always_on>true</always_on>
-                <visualize>true</visualize>
+                <visualize>false</visualize>
                 <update_rate>20</update_rate>
                 <origin xyz="0.0 0.0 0.0" rpy="0.0 0.0 0.0" />
