Commit message: Modified the sensor tags to the new Gazebo format

File: src/autobot_description/xacro/sensors.xacro (robot description, xacro)
@@ -27,10 +27,12 @@
             <material>Gazebo/Black</material>
             <gravity>true</gravity>
-            <sensor name="${name}" type="gpu_ray">
+            <sensor name="${name}" type="gpu_lidar">
                 <always_on>true</always_on>
-                <visualize>false</visualize>
+                <visualize>true</visualize>
+                <origin xyz="0.0 0.0 0.0" rpy="0.0 0.0 0.0" />
                 <update_rate>20</update_rate>
-                <origin xyz="0.0 0.0 0.0" rpy="0.0 0.0 0.0" />
-                <ray>
+                <topic>${topic}</topic>
+                <gz_frame_id>${name}</gz_frame_id>
+                <lidar>
                     <scan>
                         <horizontal>
@@ -50,20 +52,5 @@
                         <stddev>0.005</stddev>
                     </noise>
-                </ray>
-                <plugin name="${name}" filename="libgazebo_ros_ray_sensor.so">
-                    <ros>
-                        <remapping>~/out:=${topic}</remapping>
-                        <qos>
-                            <topic name="${topic}">
-                                <publisher>
-                                    <reliability>reliable</reliability>
-                                    <durability>volatile</durability>
-                                </publisher>
-                            </topic>
-                        </qos>
-                    </ros>
-                    <output_type>sensor_msgs/LaserScan</output_type>
-                    <frame_name>${name}</frame_name>
-                </plugin>
+                </lidar>
             </sensor>
         </gazebo>
